Commit message: 2.2 multiple shapes

File: src/my_r2d2/urdf/r2d2.urdf (robot description, URDF)
Before this commit: robot myfirst, 1 links, 0 joints
Links:
- added link right_leg; visual box size=0.6 0.1 0.2
Joints:
- added joint base_to_right_leg: type fixed, parent base_link, child right_leg

Commit message: 2.1.3 origins

File: src/my_r2d2/urdf/r2d2.urdf (robot description, URDF)
Before this commit: robot multipleshapes, 2 links, 1 joints
Joints:
- joint base_to_right_leg: origin (none) -> xyz=0 -0.22 0.25

Commit message: 2.1.4 materials

File: src/my_r2d2/urdf/r2d2.urdf (robot description, URDF)
Before this commit: robot origins, 2 links, 1 joints
Links:
- added link left_leg; visual box size=0.6 0.1 0.2
Joints:
- added joint base_to_left_leg: type fixed, parent base_link, child left_leg, origin xyz=0 0.22 0.25

Commit message: 2.1.5 finished model

File: src/my_r2d2/urdf/r2d2.urdf (robot description, URDF)
Before this commit: robot materials, 3 links, 2 joints
Links:
- added link box; visual box size=0.08 0.08 0.08
- added link gripper_pole; visual cylinder length=0.2 radius=0.01
- added link head; visual sphere radius=0.2
- added link left_back_wheel; visual cylinder length=0.1 radius=0.035
- added link left_base; visual box size=0.4 0.1 0.1
- added link left_front_wheel; visual cylinder length=0.1 radius=0.035
- added link left_gripper; visual mesh filename=package://urdf_tutorial/meshes/l_finger.dae
- added link left_tip; visual mesh filename=package://urdf_tutorial/meshes/l_finger_tip.dae
- added link right_back_wheel; visual cylinder length=0.1 radius=0.035
- added link right_base; visual box size=0.4 0.1 0.1
- added link right_front_wheel; visual cylinder length=0.1 radius=0.035
- added link right_gripper; visual mesh filename=package://urdf_tutorial/meshes/l_finger.dae
- added link right_tip; visual mesh filename=package://urdf_tutorial/meshes/l_finger_tip.dae
Joints:
- added joint gripper_extension: type fixed, parent base_link, child gripper_pole, origin xyz=0.19 0 0.2 rpy=0 0 0
- added joint head_swivel: type fixed, parent base_link, child head, origin xyz=0 0 0.3
- added joint left_back_wheel_joint: type fixed, parent left_base, child left_back_wheel, origin xyz=-0.133333333333 0 -0.085 rpy=0 0 0
- added joint left_base_joint: type fixed, parent left_leg, child left_base, origin xyz=0 0 -0.6
- added joint left_front_wheel_joint: type fixed, parent left_base, child left_front_wheel, origin xyz=0.133333333333 0 -0.085 rpy=0 0 0
- added joint left_gripper_joint: type fixed, parent gripper_pole, child left_gripper, origin xyz=0.2 0.01 0 rpy=0 0 0
- added joint left_tip_joint: type fixed, parent left_gripper, child left_tip
- added joint right_back_wheel_joint: type fixed, parent right_base, child right_back_wheel, origin xyz=-0.133333333333 0 -0.085 rpy=0 0 0
- added joint right_base_joint: type fixed, parent right_leg, child right_base, origin xyz=0 0 -0.6
- added joint right_front_wheel_joint: type fixed, parent right_base, child right_front_wheel, origin xyz=0.133333333333 0 -0.085 rpy=0 0 0
- added joint right_gripper_joint: type fixed, parent gripper_pole, child right_gripper, origin xyz=0.2 -0.01 0 rpy=0 0 0
- added joint right_tip_joint: type fixed, parent right_gripper, child right_tip
- added joint tobox: type fixed, parent head, child box, origin xyz=0.1814 0 0.1414

Commit message: 2.3 physical and collition properties

File: src/my_r2d2/urdf/r2d2.urdf (robot description, URDF)
Before this commit: robot visual, 16 links, 15 joints
Links:
- link base_link: mass None -> 10; geometry collision cylinder length=0.6 radius=0.2; visual cylinder length=0.6 radius=0.2
- link box: mass None -> 1; geometry collision box size=0.08 0.08 0.08; visual box size=0.08 0.08 0.08
- link gripper_pole: mass None -> 0.05; geometry collision cylinder length=0.2 radius=0.01; visual cylinder length=0.2 radius=0.01
- link head: mass None -> 2; geometry collision sphere radius=0.2; visual sphere radius=0.2
- link left_back_wheel: mass None -> 1; geometry collision cylinder length=0.1 radius=0.035; visual cylinder length=0.1 radius=0.035
- link left_base: mass None -> 10; geometry collision box size=0.4 0.1 0.1; visual box size=0.4 0.1 0.1
- link left_front_wheel: mass None -> 1; geometry collision cylinder length=0.1 radius=0.035; visual cylinder length=0.1 radius=0.035
- link left_gripper: mass None -> 0.05; geometry collision mesh filename=package://urdf_tutorial/meshes/l_finger.dae; visual mesh filename=package://urdf_tutorial/meshes/l_finger.dae
- link left_leg: mass None -> 10; geometry collision box size=0.6 0.1 0.2; visual box size=0.6 0.1 0.2
- link left_tip: mass None -> 0.05; geometry collision mesh filename=package://urdf_tutorial/meshes/l_finger_tip.dae; visual mesh filename=package://urdf_tutorial/meshes/l_finger_tip.dae
- link right_back_wheel: mass None -> 1; geometry collision cylinder length=0.1 radius=0.035; visual cylinder length=0.1 radius=0.035
- link right_base: mass None -> 10; geometry collision box size=0.4 0.1 0.1; visual box size=0.4 0.1 0.1
- link right_front_wheel: mass None -> 1; geometry collision cylinder length=0.1 radius=0.035; visual cylinder length=0.1 radius=0.035
- link right_gripper: mass None -> 0.05; geometry collision mesh filename=package://urdf_tutorial/meshes/l_finger.dae; visual mesh filename=package://urdf_tutorial/meshes/l_finger.dae
- link right_leg: mass None -> 10; geometry collision box size=0.6 0.1 0.2; visual box size=0.6 0.1 0.2
- link right_tip: mass None -> 0.05; geometry collision mesh filename=package://urdf_tutorial/meshes/l_finger_tip.dae; visual mesh filename=package://urdf_tutorial/meshes/l_finger_tip.dae
