Commit message: 3. done

File: src/my_r2d2/urdf/r2d2.urdf.xacro (robot description, xacro)
@@ -23,5 +23,14 @@
     </inertial>
   </xacro:macro>
-  <link name="base_link">
+  <!-- had to rewrite base_footprint to base, otherwise everything blew up and errored-->
+  <link name="base_footprint">
+    <visual>
+      <geometry>
+        <cylinder radius="${width*2}" length="0.01"/>
+      </geometry>
+      <material name="black"/>
+    </visual>
+  </link>
+  <link name="body_yay">
     <visual>
       <geometry>
@@ -37,16 +46,8 @@
     <xacro:default_inertial mass="10"/>
   </link>
-  <link name="base_footprint">
-    <visual>
-      <geometry>
-        <cylinder radius="${width*2}" length="0.01"/>
-      </geometry>
-      <material name="black"/>
-    </visual>
-  </link>
-  <joint name="base_footprint_to_base_link" type="fixed">
-    <parent link="base_link"/>
-    <child link="base_footprint"/>
-    <origin xyz="0 0 -${bodylen/2+wheeldiam+(wheeldiam/2+.05)}" rpy="0 0 0"/>
+  <joint name="body_yay_to_base_footprint" type="fixed">
+    <parent link="base_footprint"/>
+    <child link="body_yay"/>
+    <origin xyz="0 0 ${bodylen/2+wheeldiam+(wheeldiam/2+.05)}" rpy="0 0 0"/>
   </joint>
   <xacro:macro name="wheel" params="prefix suffix reflect">
@@ -80,5 +81,5 @@
           <box size="${leglen} 0.1 0.2"/>
         </geometry>
-        <origin xyz="0 0 -${leglen/2}" rpy="0 ${pi/2} 0"/>
+        <origin xyz="0 0 ${leglen}" rpy="0 ${pi/2} 0"/>
         <material name="white"/>
       </visual>
@@ -87,10 +88,10 @@
           <box size="${leglen} 0.1 0.2"/>
         </geometry>
-        <origin xyz="0 0 -${leglen/2}" rpy="0 ${pi/2} 0"/>
+        <origin xyz="0 0 0" rpy="0 ${pi/2} 0"/>
       </collision>
       <xacro:default_inertial mass="10"/>
     </link>
     <joint name="base_to_${prefix}_leg" type="fixed">
-      <parent link="base_link"/>
+      <parent link="base_footprint"/>
       <child link="${prefix}_leg"/>
       <origin xyz="0 ${reflect*(width+.02)} 0.25" />
@@ -113,5 +114,5 @@
       <parent link="${prefix}_leg"/>
       <child link="${prefix}_base"/>
-      <origin xyz="0 0 ${-leglen}" />
+      <origin xyz="0 0 0" />
     </joint>
     <xacro:wheel prefix="${prefix}" suffix="front" reflect="1"/>
@@ -121,5 +122,5 @@
   <xacro:leg prefix="left" reflect="1" />
   <joint name="gripper_extension" type="prismatic">
-    <parent link="base_link"/>
+    <parent link="base_footprint"/>
     <child link="gripper_pole"/>
     <limit effort="1000.0" lower="-${width*2-.02}" upper="0" velocity="0.5"/>
@@ -201,8 +202,8 @@
   </link>
   <joint name="head_swivel" type="continuous">
-    <parent link="base_link"/>
+    <parent link="base_footprint"/>
     <child link="head"/>
     <axis xyz="0 0 1"/>
-    <origin xyz="0 0 ${bodylen/2}"/>
+    <origin xyz="0 0 ${bodylen+width}"/>
   </joint>
   <link name="box">
