Commit message: 2.5 added black lens

File: src/my_r2d2/urdf/r2d2-from-xacro.urdf (robot description, URDF)
Before this commit: robot macroed, 16 links, 15 joints
Links:
- added link lens, mass 1; collision cylinder length=0.015 radius=0.03; visual cylinder length=0.015 radius=0.03
Joints:
- added joint lens_to_box: type fixed, parent box, child lens, origin xyz=0 0 0 rpy=0 1.57075 0

File: src/my_r2d2/urdf/r2d2.urdf.xacro (robot description, xacro)
@@ -213,3 +213,24 @@
     <origin xyz="${.707*width+0.04} 0 ${.707*width}"/>
   </joint>
+  <link name="lens">
+    <visual>
+      <geometry>
+        <cylinder radius="0.03" length="0.015" />
+      </geometry>
+      <material name="black"/>
+      <origin xyz="0 0 0" />
+    </visual>
+    <collision>
+      <geometry>
+        <cylinder radius="0.03" length="0.015" />
+      </geometry>
+      <origin xyz="0 0 0"/>
+    </collision>
+    <xacro:default_inertial mass="1"/>
+  </link>
+  <joint name="lens_to_box" type="fixed">
+    <parent link="box"/>
+    <child link="lens"/>
+    <origin xyz="0 0 0" rpy="0 ${pi/2} 0"/>
+  </joint>
 </robot>

Commit message: 3. added base_footprint

File: src/my_r2d2/urdf/r2d2-from-xacro.urdf (robot description, URDF)
Before this commit: robot macroed, 17 links, 16 joints
Links:
- added link base_footprint; visual cylinder length=0.01 radius=0.4
Joints:
- added joint base_footprint_to_base_link: type fixed, parent base_link, child base_footprint, origin xyz=0 0 -0.455 rpy=0 0 0

File: src/my_r2d2/urdf/r2d2.urdf.xacro (robot description, xacro)
@@ -37,4 +37,17 @@
     <xacro:default_inertial mass="10"/>
   </link>
+  <link name="base_footprint">
+    <visual>
+      <geometry>
+        <cylinder radius="${width*2}" length="0.01"/>
+      </geometry>
+      <material name="black"/>
+    </visual>
+  </link>
+  <joint name="base_footprint_to_base_link" type="fixed">
+    <parent link="base_link"/>
+    <child link="base_footprint"/>
+    <origin xyz="0 0 -${bodylen/2+wheeldiam+(wheeldiam/2+.05)}" rpy="0 0 0"/>
+  </joint>
   <xacro:macro name="wheel" params="prefix suffix reflect">
     <link name="${prefix}_${suffix}_wheel">

Commit message: add some issue with missing files

File: src/my_r2d2/urdf/r2d2-from-xacro.urdf (robot description, URDF)
Before this commit: robot macroed, 18 links, 17 joints
Links:
- added link eye
Joints:
- added joint eye_to_lens: type fixed, parent lens, child eye, origin xyz=0 0 0 rpy=0 1.57075 0
